File: keyboards/maddykb/madosplit/design/output/pcbs/_autosave-MadoSplit.kicad_pcb (KiCad board)
At the start: 2 copper layers, 310.9 x 110.8 mm, 132 parts

Commit message: done wiring both board, missing resistors
Connections:
- REF** pad 1: (no net) -> GND
- REF** pad 2: (no net) -> P0
- REF** pad 3: (no net) -> P1
- REF** pad 4: (no net) -> VCC
- TRRS1 pad 2: GND -> P0
- TRRS1 pad 3: P0 -> P1
Routing:
- net P1: track 0.00 -> 54.1 mm
- net GND: track 88.7 -> 102.6 mm
- net P0: track 55.5 -> 59.6 mm
Changed lines of the file:
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@@
 			(layers "*.Cu" "*.Mask")
 			(remove_unused_layers no)
+			(net 72 "GND")
 		)
 		(pad "2" thru_hole oval
@@
 			(layers "*.Cu" "*.Mask")
 			(remove_unused_layers no)
+			(net 78 "P0")
 		)
 		(pad "3" thru_hole oval
@@
 			(layers "*.Cu" "*.Mask")
 			(remove_unused_layers no)
+			(net 77 "P1")
 		)
 		(pad "4" thru_hole oval
@@
 			(layers "*.Cu" "*.Mask")
 			(remove_unused_layers no)
+			(net 74 "VCC")
 		)
 		(model "${SCOTTOKEEBS_KICAD}/3dmodels/ScottoKeebs_Components.3dshapes/TRRS_PJ-320A.step"
@@
 			(layers "*.Cu" "*.Mask")
 			(remove_unused_layers no)
-			(net 72 "GND")
+			(net 78 "P0")
 		)
 		(pad "3" thru_hole oval
@@
 			(layers "*.Cu" "*.Mask")
 			(remove_unused_layers no)
-			(net 78 "P0")
+			(net 77 "P1")
 		)
 		(pad "4" thru_hole oval
@@
 		(tags "SOD-123")
 		(property "Reference" "D29"
-			(at 0 2.000002 360)
+			(at 0 2.000002 0)
 			(layer "B.SilkS")
 			(hide yes)
@@
 		)
 		(property "Value" ""
-			(at 0.000001 -2.099999 360)
+			(at 0.000001 -2.099999 0)
 			(layer "B.Fab")
 			(effects
@@
 		)
 		(fp_text user "${REFERENCE}"
-			(at 0 2.000002 360)
+			(at 0 2.000002 0)
 			(layer "B.Fab")
 			(effects
@@
 	)
 	(segment
+		(start 262.5 41.35)
+		(end 266.28 37.57)
+		(width 0.25)
+		(layer "F.Cu")
+		(net 72)
+	)
+	(segment
 		(start 224.65 53.1)
 		(end 224.65 39.6)
@@
 	)
 	(segment
-		(start 257.6 42.05)
-		(end 257.6 55.85)
+		(start 259.55 57.8)
+		(end 263.6 53.75)
 		(width 0.25)
 		(layer "F.Cu")
@@
 	)
 	(segment
-		(start 257.6 55.85)
-		(end 259.55 57.8)
+		(start 262.5 42.85)
+		(end 262.5 41.35)
+		(width 0.25)
+		(layer "F.Cu")
+		(net 72)
+	)
+	(segment
+		(start 263.6 53.75)
+		(end 263.6 43.95)
+		(width 0.25)
+		(layer "F.Cu")
+		(net 72)
+	)
+	(segment
+		(start 263.6 43.95)
+		(end 262.5 42.85)
 		(width 0.25)
 		(layer "F.Cu")
@@
 	)
 	(segment
+		(start 226.7 41.65)
+		(end 222.62 37.57)
+		(width 0.25)
+		(layer "F.Cu")
+		(net 72)
+	)
+	(segment
 		(start 259.55 57.8)
 		(end 259.55 64)
@@
 	)
 	(segment
-		(start 257.9 41.75)
-		(end 257.6 42.05)
+		(start 224.65 39.6)
+		(end 222.62 37.57)
 		(width 0.25)
 		(layer "F.Cu")
@@
 	)
 	(segment
-		(start 224.65 39.6)
-		(end 222.62 37.57)
+		(start 226.7 42.9)
+		(end 226.7 41.65)
 		(width 0.25)
 		(layer "F.Cu")
@@
 	)
 	(segment
-		(start 263.625 42.765)
+		(start 264.6 41.79)
 		(end 266.28 40.11)
 		(width 0.25)
@@
 	)
 	(segment
-		(start 225.65 55.45)
-		(end 224.2 54)
+		(start 264.6 56.45)
+		(end 264.6 41.79)
 		(width 0.25)
 		(layer "F.Cu")
@@
 	)
 	(segment
-		(start 224.2 54)
-		(end 224.2 41.69)
+		(start 263.25 57.8)
+		(end 264.6 56.45)
 		(width 0.25)
 		(layer "F.Cu")
@@
 	)
 	(segment
-		(start 263.25 57.8)
-		(end 263.625 57.425)
+		(start 225.65 55.45)
+		(end 224.2 54)
 		(width 0.25)
 		(layer "F.Cu")
@@
 	)
 	(segment
-		(start 263.625 57.425)
-		(end 263.625 42.765)
+		(start 224.2 54)
+		(end 224.2 41.69)
 		(width 0.25)
 		(layer "F.Cu")
@@
 	)
 	(segment
+		(start 226.8787 33.3787)
+		(end 209.0313 33.3787)
+		(width 0.25)
+		(layer "F.Cu")
+		(net 77)
+	)
+	(segment
+		(start 278.49 32)
+		(end 281.52 35.03)
+		(width 0.25)
+		(layer "F.Cu")
+		(net 77)
+	)
+	(segment
+		(start 231.3 37.8)
+		(end 226.8787 33.3787)
+		(width 0.25)
+		(layer "F.Cu")
+		(net 77)
+	)
+	(segment
+		(start 263.65 32)
+		(end 278.49 32)
+		(width 0.25)
+		(layer "F.Cu")
+		(net 77)
+	)
+	(segment
 		(start 257.9 37.75)
-		(end 262.85 32.8)
+		(end 263.65 32)
 		(width 0.25)
 		(layer "F.Cu")
-		(net 78)
+		(net 77)
 	)
 	(segment
-		(start 211.95 33)
-		(end 207.38 37.57)
+		(start 209.0313 33.3787)
+		(end 207.38 35.03)
+		(width 0.25)
+		(layer "F.Cu")
+		(net 77)
+	)
+	(segment
+		(start 231 37.75)
+		(end 230.65 37.75)
+		(width 0.25)
+		(layer "B.Cu")
+		(net 77)
+	)
+	(segment
+		(start 230.65 37.75)
+		(end 230.6 37.8)
+		(width 0.25)
+		(layer "B.Cu")
+		(net 77)
+	)
+	(segment
+		(start 257.9 40.1)
+		(end 265 33)
 		(width 0.25)
 		(layer "F.Cu")
@@
 	)
 	(segment
-		(start 225.6 33)
-		(end 211.95 33)
+		(start 231.3 40.55)
+		(end 224.5787 33.8287)
 		(width 0.25)
 		(layer "F.Cu")
@@
 	)
 	(segment
-		(start 276.75 32.8)
-		(end 281.52 37.57)
+		(start 257.9 41.75)
+		(end 257.9 40.1)
 		(width 0.25)
 		(layer "F.Cu")
@@
 	)
 	(segment
-		(start 262.85 32.8)
-		(end 276.75 32.8)
+		(start 211.1213 33.8287)
+		(end 207.38 37.57)
 		(width 0.25)
 		(layer "F.Cu")
@@
 	)
 	(segment
-		(start 230.35 37.75)
-		(end 225.6 33)
+		(start 231.3 41.8)
+		(end 231.3 40.55)
 		(width 0.25)
 		(layer "F.Cu")
@@
 	)
 	(segment
-		(start 231 37.75)
-		(end 230.35 37.75)
+		(start 276.95 33)
+		(end 281.52 37.57)
 		(width 0.25)
 		(layer "F.Cu")
@@
 	)
 	(segment
-		(start 231 37.75)
-		(end 230.65 37.75)
+		(start 265 33)
+		(end 276.95 33)
 		(width 0.25)
-		(layer "B.Cu")
+		(layer "F.Cu")
 		(net 78)
 	)
 	(segment
-		(start 230.65 37.75)
-		(end 230.6 37.8)
+		(start 224.5787 33.8287)
+		(end 211.1213 33.8287)
 		(width 0.25)
-		(layer "B.Cu")
+		(layer "F.Cu")
 		(net 78)
 	)
