File: keyboards/maddykb/madosplit/design/output/pcbs/MadoSplit.kicad_pcb (KiCad board)
At the start: 2 copper layers, 310.9 x 110.8 mm, 132 parts

Commit message: MadoSplit PCB finish
Parts:
- added REF**: Resistor_0402, ScottoKeebs_Components:Resistor_0402, B.Cu at (259.5, 45.0)
- added REF**: Resistor_0402, ScottoKeebs_Components:Resistor_0402, B.Cu at (230.5, 45.0)
- added REF**: Resistor_0402, ScottoKeebs_Components:Resistor_0402, B.Cu at (259.5, 46.5)
- added REF**: Resistor_0402, ScottoKeebs_Components:Resistor_0402, B.Cu at (230.5, 46.5)
- TRRS1: value TRRS-PJ-320A-dual -> TRRS_PJ-320A; footprint TRRS-PJ-320A-dual -> ScottoKeebs_Components:TRRS_PJ-320A; moved to F.Cu
- moved TRRS1 2.10 mm to (260.0, 31.6), turned to 0 degrees
Connections:
- REF** pad 1: (no net) -> GND
- REF** pad 2: (no net) -> P0
- REF** pad 3: (no net) -> P1
- REF** pad 4: (no net) -> VCC
- TRRS1 pad 2: GND -> P0
- TRRS1 pad 3: P0 -> P1
Routing:
- net P1: track 0.00 -> 107.8 mm, vias 0 -> 2
- net P0: track 55.5 -> 79.0 mm, vias 0 -> 2
- net VCC: track 81.2 -> 99.2 mm
- net GND: track 88.7 -> 89.5 mm
