File: keyboards/maddykb/madosplit/design/output/pcbs/MadoSplit.kicad_pcb (KiCad board)
At the start: 2 copper layers, 310.9 x 110.8 mm, 140 parts

Commit message: Debugged Firmware Case + gasket STL
Parts:
- removed the B1 at (261.4, 60.9)
- removed G*** (x2): LOGO, Graphics:Crewmate
- removed G*** (x2): LOGO, Graphics:MadoSplit
- removed the MCU1 at (273.9, 49.0)
- removed the OLED1 at (268.0, 70.0)
- removed the OLED1 at (209.0, 70.0)
- removed RES1, RES2, RES3, RES4: R_0402_1005Metric, Resistor_SMD:R_0402_1005Metric
- removed TRRS2: TRRS_PJ-320A, ScottoKeebs_Components:TRRS_PJ-320A
- removed the _1 at (364.9, 32.4)
- removed the _2 at (360.9, 111.6)
- removed the _3 at (289.9, 109.0)
- removed the _4 at (260.4, 52.4)
- added OLED1: OLED, lib:OLED_headers, F.Cu at (209.0, 70.0)
- D1, D10, D11, D12, D13, D14, D15, D16, D17, D18, D19, D2, D20, D21, D22, D23, D24, D25, D26, D27, D28, D29, D3, D30, D31, D32, D33, D34, D35, D36, D37, D38, D39, D4, D40, D41, D42, D43, D44, D45, D46, D47, D48, D49, D5, D50, D51, D52, D53, D54, D55, D56, D57, D58, D6, D7, D8, D9: footprint ScottoKeebs_Components:Diode_SOD-123 -> ComboDiode; moved to F.Cu
- S1, S10, S11, S12, S13, S14, S15, S16, S17, S18, S19, S2, S20, S21, S22, S23, S24, S25, S26, S27, S28, S3, S30, S31, S32, S33, S34, S35, S36, S37, S38, S39, S4, S40, S41, S42, S43, S44, S45, S46, S47, S48, S49, S5, S50, S51, S52, S53, S54, S55, S56, S57, S6, S7, S8, S9: footprint ScottoKeebs_Hotswap:Hotswap_Choc_V1V2_1.00u -> PG1350
- S29, S58: footprint ScottoKeebs_Hotswap:Hotswap_Choc_V1V2_1.50u -> PG1350
- TRRS1: value TRRS_PJ-320A -> TRRS-PJ-320A-dual; footprint ScottoKeebs_Components:TRRS_PJ-320A -> TRRS-PJ-320A-dual
- moved D29 17.4 mm to (216.8, 116.0), turned to 155 degrees
- moved D30 8.10 mm to (393.0, 95.0), turned to -270 degrees
- moved D31 8.10 mm to (393.0, 77.0), turned to -270 degrees
- moved D32 8.10 mm to (393.0, 59.0), turned to -270 degrees
- moved D33 8.10 mm to (393.0, 41.0), turned to -270 degrees
- moved D34 8.10 mm to (374.0, 93.0), turned to -270 degrees
- moved D35 8.10 mm to (374.0, 75.0), turned to -270 degrees
- moved D36 8.10 mm to (374.0, 57.0), turned to -270 degrees
- moved D37 8.10 mm to (374.0, 39.0), turned to -270 degrees
- moved D38 8.10 mm to (355.0, 87.0), turned to -270 degrees
- moved D39 8.10 mm to (355.0, 69.0), turned to -270 degrees
- moved D40 8.10 mm to (355.0, 51.0), turned to -270 degrees
- moved D41 8.10 mm to (355.0, 33.0), turned to -270 degrees
- moved D42 8.10 mm to (336.0, 84.5), turned to -270 degrees
- moved D43 8.10 mm to (336.0, 66.5), turned to -270 degrees
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Connections:
- TRRS1 pad 2: P0 -> GND
- TRRS1 pad 3: P1 -> P0
Routing:
- net P19: track 530.4 -> 0.00 mm
- net P18: track 490.3 -> 0.00 mm
- net P15: track 460.9 -> 0.00 mm
- net P14: track 418.5 -> 0.00 mm
- net P16: track 373.8 -> 0.00 mm
- net P10: track 310.7 -> 0.00 mm, vias 2 -> 0
- net P7: track 284.2 -> 0.00 mm, vias 21 -> 0
- net P6: track 250.7 -> 0.00 mm, vias 21 -> 0
- net P9: track 246.7 -> 0.00 mm, vias 12 -> 0
- net P5: track 234.1 -> 0.00 mm, vias 21 -> 0
- net P4: track 232.8 -> 0.00 mm
- net P1: track 107.8 -> 0.00 mm, vias 2 -> 0
- net VCC: track 99.2 -> 0.00 mm
- net GND: track 89.5 -> 0.00 mm
- net P0: track 79.0 -> 0.00 mm, vias 2 -> 0
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Other:
- board size 310.9 x 110.8 mm -> 145.8 x 110.8 mm
- net class Default added: clearance 0.2, trace_width 0.25, via_dia 0.8, via_drill 0.4
