File: keyboards/maddykb/madosplit/design/output/pcbs/MadoSplitFinal.kicad_pcb (KiCad board)
At the start: 2 copper layers, 310.9 x 110.8 mm, 140 parts

Commit message: Started madosplitV2 and fixed some layout issues on V1
Connections:
- OLED1 pad 3: P2 -> P3 (x2)
- OLED1 pad 4: P3 -> P2 (x2)
Routing:
- net P4: track 232.8 -> 252.6 mm
- net P3: track 57.9 -> 47.6 mm
- net GND: track 89.5 -> 86.7 mm
Changed lines of the file:
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@@
 			(layers "*.Cu" "*.Mask")
 			(remove_unused_layers no)
-			(net 79 "P2")
+			(net 80 "P3")
 		)
 		(pad "4" thru_hole oval
@@
 			(layers "*.Cu" "*.Mask")
 			(remove_unused_layers no)
-			(net 80 "P3")
+			(net 79 "P2")
 		)
 		(model "${SCOTTOKEEBS_KICAD}/3dmodels/ScottoKeebs_Components.3dshapes/OLED_128x32.step"
@@
 			(layers "*.Cu" "*.Mask")
 			(remove_unused_layers no)
-			(net 79 "P2")
+			(net 80 "P3")
 		)
 		(pad "4" thru_hole oval
@@
 			(layers "*.Cu" "*.Mask")
 			(remove_unused_layers no)
-			(net 80 "P3")
+			(net 79 "P2")
 		)
 		(model "${SCOTTOKEEBS_KICAD}/3dmodels/ScottoKeebs_Components.3dshapes/OLED_128x32.step"
@@
 	)
 	(segment
+		(start 289.9 33.85)
+		(end 282.7213 41.0287)
+		(width 0.25)
+		(layer "B.Cu")
+		(net 68)
+	)
+	(segment
 		(start 169.5 28.85)
 		(end 172 31.35)
@@
 	)
 	(segment
+		(start 282.7213 49.0687)
+		(end 281.52 50.27)
+		(width 0.25)
+		(layer "B.Cu")
+		(net 68)
+	)
+	(segment
 		(start 133.313604 31.35)
 		(end 134 31.35)
@@
 	)
 	(segment
+		(start 282.7213 41.0287)
+		(end 282.7213 49.0687)
+		(width 0.25)
+		(layer "B.Cu")
+		(net 68)
+	)
+	(segment
 		(start 203 45.89)
 		(end 207.38 50.27)
@@
 	)
 	(segment
-		(start 273.199999 73)
-		(end 277.8 68.399999)
-		(width 0.25)
-		(layer "F.Cu")
-		(net 72)
-	)
-	(segment
 		(start 264.27099 37.57)
 		(end 266.28 37.57)
@@
 	)
 	(segment
-		(start 268.55 73)
-		(end 273.199999 73)
-		(width 0.25)
-		(layer "F.Cu")
-		(net 72)
-	)
-	(segment
 		(start 226.7 41.65)
 		(end 222.62 37.57)
@@
 	)
 	(segment
-		(start 259.55 57.8)
-		(end 259.55 64)
-		(width 0.25)
-		(layer "F.Cu")
-		(net 72)
-	)
-	(segment
 		(start 224.95 68.4)
 		(end 229.35 64)
@@
 	)
 	(segment
-		(start 259.55 64)
-		(end 268.55 73)
-		(width 0.25)
-		(layer "F.Cu")
-		(net 72)
-	)
-	(segment
 		(start 224.65 39.6)
 		(end 222.62 37.57)
@@
 	)
 	(segment
+		(start 277.8 68.399999)
+		(end 277.8 46.37)
+		(width 0.2)
+		(layer "B.Cu")
+		(net 72)
+	)
+	(segment
+		(start 277.8 46.37)
+		(end 281.52 42.65)
+		(width 0.2)
+		(layer "B.Cu")
+		(net 72)
+	)
+	(segment
 		(start 264.6 41.79)
 		(end 266.28 40.11)
@@
 	)
 	(segment
-		(start 272.719995 68.400001)
-		(end 272.719995 53.990005)
-		(width 0.25)
+		(start 270.179995 68.4)
+		(end 270.179995 56.530005)
+		(width 0.2)
 		(layer "F.Cu")
 		(net 79)
 	)
 	(segment
-		(start 272.719995 53.990005)
-		(end 281.52 45.19)
-		(width 0.25)
+		(start 211.18 68.4)
+		(end 211.18 48.99)
+		(width 0.2)
 		(layer "F.Cu")
 		(net 79)
 	)
 	(segment
-		(start 213.72 51.53)
-		(end 207.38 45.19)
-		(width 0.25)
-		(layer "B.Cu")
+		(start 270.179995 56.530005)
+		(end 281.52 45.19)
+		(width 0.2)
+		(layer "F.Cu")
 		(net 79)
 	)
 	(segment
-		(start 213.72 68.4)
-		(end 213.72 51.53)
-		(width 0.25)
-		(layer "B.Cu")
+		(start 211.18 48.99)
+		(end 207.38 45.19)
+		(width 0.2)
+		(layer "F.Cu")
 		(net 79)
 	)
 	(segment
-		(start 277.6 72.6)
-		(end 279.8 70.4)
-		(width 0.25)
-		(layer "B.Cu")
-		(net 80)
-	)
-	(segment
-		(start 211.18 51.53)
-		(end 207.38 47.73)
-		(width 0.25)
-		(layer "B.Cu")
-		(net 80)
-	)
-	(segment
-		(start 270.179995 68.4)
-		(end 274.379995 72.6)
-		(width 0.25)
-		(layer "B.Cu")
-		(net 80)
-	)
-	(segment
-		(start 274.379995 72.6)
-		(end 277.6 72.6)
-		(width 0.25)
-		(layer "B.Cu")
+		(start 272.719995 56.530005)
+		(end 281.52 47.73)
+		(width 0.2)
+		(layer "F.Cu")
 		(net 80)
 	)
 	(segment
-		(start 279.8 49.45)
-		(end 281.52 47.73)
-		(width 0.25)
-		(layer "B.Cu")
+		(start 272.719995 68.400001)
+		(end 272.719995 56.530005)
+		(width 0.2)
+		(layer "F.Cu")
 		(net 80)
 	)
 	(segment
-		(start 279.8 70.4)
-		(end 279.8 49.45)
-		(width 0.25)
+		(start 213.72 54.07)
+		(end 207.38 47.73)
+		(width 0.2)
 		(layer "B.Cu")
 		(net 80)
 	)
 	(segment
-		(start 211.18 68.4)
-		(end 211.18 51.53)
-		(width 0.25)
+		(start 213.72 68.4)
+		(end 213.72 54.07)
+		(width 0.2)
 		(layer "B.Cu")
 		(net 80)
